File: k1921vg015_devboard.kicad_sch (KiCad schematic)
At the start: 46 parts, among them J1 Conn_02x25_Odd_Even, J2 Conn_02x25_Odd_Even, J3 Conn_02x06_Odd_Even, J4 Conn_02x01, J7 USB_C_Receptacle_USB2.0_16P, U1 AMS1117-3.3, U2 TL432DBZ, Y2 Crystal, Y3 Crystal

Commit message: add silkscreen
Parts:
- added D4, D5: LED, LED_SMD:LED_1206_3216Metric_Pad1.42x1.75mm_HandSolder, symbol Device:LED
- added R16, R17: 1k, Resistor_SMD:R_0805_2012Metric_Pad1.20x1.40mm_HandSolder, symbol Device:R
Connections:
- net +3V3: now also J2.7 (Pin_7), R17.1
- net 5V: now also J2.5 (Pin_5), R16.1
- net GND: now also J2.6 (Pin_6), J2.8 (Pin_8), D4.1 (K)
- net PA0: now also D5.1 (K)
- new net: D4.2 (A), R16.2
- new net: D5.2 (A), R17.2
